File: gps_board/gpsSchematic.brd (EAGLE design)
At the start: 49.5 x 40.6 mm, 64 parts, among them J1 Qwiic Right Angle, J2 1050170001, J4 BOOT, U1 UBLOX_SAM_M8Q-0-10

Commit message: Workedd on powerboard
Parts:
- moved J2 2.03 mm to (64.3, 59.7)
Routing:
- net SCL: track 82.3 -> 84.7 mm
- net SDA: track 74.9 -> 77.0 mm
- net 3.3V: track 157.2 -> 159.3 mm
Changed lines of the file:
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@@
 </element>
 <element name="U$31" library="JP2" package="JP20" value="" x="51.0286" y="51.4858" smashed="yes"/>
-<element name="J2" library="1050170001" package="MOLEX_1050170001" value="1050170001" x="62.23" y="59.69" smashed="yes" rot="R90">
-<attribute name="AVAILABILITY" value="Unavailable" x="62.23" y="59.69" size="1.778" layer="27" rot="R90" display="off"/>
-<attribute name="DESCRIPTION" value=" Conn.; Data; USB; Recept.; Micro; B Type; Bottom Mount, SMT, with Solder Tabs, Lead-Free " x="62.23" y="59.69" size="1.778" layer="27" rot="R90" display="off"/>
-<attribute name="MF" value="Molex" x="62.23" y="59.69" size="1.778" layer="27" rot="R90" display="off"/>
-<attribute name="MP" value="1050170001" x="62.23" y="59.69" size="1.778" layer="27" rot="R90" display="off"/>
-<attribute name="NAME" x="58.58976875" y="55.37973125" size="1.27008125" layer="25" rot="R90"/>
-<attribute name="PACKAGE" value="None" x="62.23" y="59.69" size="1.778" layer="27" rot="R90" display="off"/>
-<attribute name="PRICE" value="None" x="62.23" y="59.69" size="1.778" layer="27" rot="R90" display="off"/>
-<attribute name="VALUE" x="66.48266875" y="55.3773" size="1.2708" layer="27" rot="R90"/>
+<element name="J2" library="1050170001" package="MOLEX_1050170001" value="1050170001" x="64.262" y="59.69" smashed="yes" rot="R90">
+<attribute name="AVAILABILITY" value="Unavailable" x="64.262" y="59.69" size="1.778" layer="27" rot="R90" display="off"/>
+<attribute name="DESCRIPTION" value=" Conn.; Data; USB; Recept.; Micro; B Type; Bottom Mount, SMT, with Solder Tabs, Lead-Free " x="64.262" y="59.69" size="1.778" layer="27" rot="R90" display="off"/>
+<attribute name="MF" value="Molex" x="64.262" y="59.69" size="1.778" layer="27" rot="R90" display="off"/>
+<attribute name="MP" value="1050170001" x="64.262" y="59.69" size="1.778" layer="27" rot="R90" display="off"/>
+<attribute name="NAME" x="60.62176875" y="55.37973125" size="1.27008125" layer="25" rot="R90"/>
+<attribute name="PACKAGE" value="None" x="64.262" y="59.69" size="1.778" layer="27" rot="R90" display="off"/>
+<attribute name="PRICE" value="None" x="64.262" y="59.69" size="1.778" layer="27" rot="R90" display="off"/>
+<attribute name="VALUE" x="68.51466875" y="55.3773" size="1.2708" layer="27" rot="R90"/>
 </element>
 <element name="JP4" library="pinhead" package="1X02" value="" x="24.384" y="63.627" smashed="yes" rot="R90">
@@
 <wire x1="55.88" y1="57.15" x2="58.42" y2="57.15" width="0.254" layer="1"/>
 <wire x1="58.42" y1="57.15" x2="58.42" y2="57.785" width="0.254" layer="1"/>
-<wire x1="59.025" y1="58.39" x2="59.88" y2="58.39" width="0.254" layer="1"/>
+<wire x1="59.025" y1="58.39" x2="61.912" y2="58.39" width="0.254" layer="1"/>
 <wire x1="58.42" y1="57.785" x2="59.025" y2="58.39" width="0.254" layer="1"/>
 </signal>
@@
 <wire x1="57.15" y1="60.7568" x2="52.4256" y2="60.7568" width="0.254" layer="1"/>
 <contactref element="J2" pad="2"/>
-<wire x1="60.8344" y1="59.37426875" x2="60.8344" y2="59.5644" width="0.254" layer="1"/>
-<wire x1="60.8344" y1="59.5644" x2="60.96" y2="59.69" width="0.254" layer="1"/>
-<wire x1="59.88" y1="59.04" x2="60.50013125" y2="59.04" width="0.254" layer="1"/>
-<wire x1="60.50013125" y1="59.04" x2="60.8344" y2="59.37426875" width="0.254" layer="1"/>
-<wire x1="60.96" y1="59.69" x2="60.96" y2="63.5" width="0.254" layer="1"/>
-<wire x1="60.96" y1="63.5" x2="58.42" y2="63.5" width="0.254" layer="1"/>
+<wire x1="63.119" y1="59.309" x2="62.85" y2="59.04" width="0.254" layer="1"/>
+<wire x1="61.912" y1="59.04" x2="62.85" y2="59.04" width="0.254" layer="1"/>
+<wire x1="63.119" y1="59.309" x2="63.119" y2="63.5" width="0.254" layer="1"/>
+<wire x1="63.119" y1="63.5" x2="58.42" y2="63.5" width="0.254" layer="1"/>
 <wire x1="58.42" y1="63.5" x2="57.15" y2="62.23" width="0.254" layer="1"/>
 <wire x1="57.15" y1="62.23" x2="57.15" y2="60.7568" width="0.254" layer="1"/>
@@
 <wire x1="43.18" y1="39.37" x2="43.18" y2="43.18" width="0.254" layer="1"/>
 <contactref element="J2" pad="3"/>
-<wire x1="52.197" y1="59.563" x2="50.9016" y2="58.2676" width="0.254" layer="1"/>
-<wire x1="52.197" y1="59.563" x2="52.324" y2="59.69" width="0.254" layer="1"/>
-<wire x1="52.324" y1="59.69" x2="59.88" y2="59.69" width="0.254" layer="1"/>
+<wire x1="52.324" y1="59.69" x2="50.9016" y2="58.2676" width="0.254" layer="1"/>
+<wire x1="52.324" y1="59.69" x2="61.912" y2="59.69" width="0.254" layer="1"/>
 </signal>
 <signal name="!RESET">
